File: examples/lef-mega-testboard/schematic/lef-mega-testboard.kicad_sch (KiCad schematic)
At the start: 0 parts

Commit message: Fixed 4 led function Refactored code Updated schematic
Parts:
- added A1: Arduino_Mega2560_R3_Shield, PCM_arduino-library:Arduino_Mega2560_R3_Shield, symbol arduino-library:Arduino_Mega2560_R3_Shield
- added BZ1: Buzzer, symbol Device:Buzzer
- added D1, D3, D4, D5: LED, symbol Device:LED
- added D2: WS2812B, LED_SMD:LED_WS2812B_PLCC4_5.0x5.0mm_P3.2mm, symbol LED:WS2812B
- added R1, R2, R3, R4: 470, symbol Device:R
- added RV1: R_Potentiometer, symbol Device:R_Potentiometer
- added SW1: RotaryEncoder_Switch, symbol Device:RotaryEncoder_Switch
- added U1: DS18B20, Package_TO_SOT_THT:TO-92_Inline, symbol Sensor_Temperature:DS18B20
- added U2: DHT11, Sensor:Aosong_DHT11_5.5x12.0_P2.54mm, symbol Sensor:DHT11
Connections:
- new net: D3.2 (A), R2.2
- new net: D4.2 (A), R3.2
- new net: D5.2 (A), R4.2
- new net: D1.2 (A), R1.2
- new net +5V: A1.5V1 (5V), RV1.3
- new net GND: A1.GND6 (GND), BZ1.2 (-), D1.1 (K), D3.1 (K), D4.1 (K), D5.1 (K), RV1.1

Commit message: Schematic
Connections:
- net at R3.1: now also A1.A14
- net at R4.1: now also A1.A15
- net at R2.1: now also A1.A13
- net at R1.1: now also A1.A12
Other:
- moved on the sheet: D1, D3, D4, D5, R1, R2, R3, R4

Commit message: Updated schematic
Parts:
- removed D2: WS2812B, LED_SMD:LED_WS2812B_PLCC4_5.0x5.0mm_P3.2mm, symbol LED:WS2812B
- removed U1: DS18B20, Package_TO_SOT_THT:TO-92_Inline, symbol Sensor_Temperature:DS18B20
- removed U2: DHT11, Sensor:Aosong_DHT11_5.5x12.0_P2.54mm, symbol Sensor:DHT11
- added D6: LED_Dual_AAK, LED_THT:LED_D5.0mm-4_RGB, symbol Device:LED_Dual_AAK
- added J1: HD44780, Display:HY1602E, symbol Connector_Generic:Conn_01x16
- added R5, R6: 470, Resistor_THT:R_Axial_DIN0309_L9.0mm_D3.2mm_P15.24mm_Horizontal, symbol Device:R
- added RV2: 10K, Potentiometer_THT:Potentiometer_Alpha_RD902F-40-00D_Dual_Vertical, symbol Device:R_Potentiometer
- added SW2, SW3, SW4: SW_Push, Button_Switch_THT:SW_PUSH_6mm, symbol Switch:SW_Push
- BZ1: footprint (none) -> Buzzer_Beeper:Buzzer_12x9.5RM7.6
- D1, D3, D4, D5: footprint (none) -> LED_THT:LED_D5.0mm
- R1, R2, R3, R4: footprint (none) -> Resistor_THT:R_Axial_DIN0309_L9.0mm_D3.2mm_P15.24mm_Horizontal
- RV1: value R_Potentiometer -> 10k; footprint (none) -> Potentiometer_THT:Potentiometer_Alpha_RD902F-40-00D_Dual_Vertical
- SW1: footprint (none) -> Rotary_Encoder:RotaryEncoder_Alps_EC12E-Switch_Vertical_H20mm_CircularMountingHoles
Connections:
- net +5V: now also J1.2 (Pin_2), RV2.3
- net GND: now also J1.1 (Pin_1), R5.2, RV2.1, SW2.2, SW3.2, SW4.2
- net at BZ1.1 (+): now also R6.1
- net LED2: now reaches A1.A14, R3.1
- net LED1: now reaches A1.A15, R4.1
- net LED3: now reaches A1.A13, R2.1
- net LED4: now reaches A1.A12, R1.1
- net Pot: now reaches RV1.2
- net Pot: now also A1.A8
- net LD7: now reaches A1.A1
- net LD7: now also J1.14 (Pin_14)
- net LED Green: now reaches A1.A10
- net LED Green: now also D6.1 (A1)
- net LED Red: now reaches A1.A11
- net LED Red: now also D6.2 (A2)
- net LD6: now reaches A1.A2
- net LD6: now also J1.13 (Pin_13)
- net LD5: now reaches A1.A3
- net LD5: now also J1.12 (Pin_12)
- net LD4: now reaches A1.A4
- net LD4: now also J1.11 (Pin_11)
- net E: now reaches A1.A5
- net E: now also J1.6 (Pin_6)
- net RW: now reaches A1.A6
- net RW: now also J1.5 (Pin_5)
- net RS: now reaches A1.A7
- net RS: now also J1.4 (Pin_4)
- net Buzzer: now reaches A1.A9
- net Buzzer: now also R6.2
- new net: D6.3 (K), R5.1
- new net BL+: J1.15 (Pin_15)
- new net BL-: J1.16 (Pin_16)
- new net LD0: J1.7 (Pin_7)
- new net LD1: J1.8 (Pin_8)
- new net LD2: J1.9 (Pin_9)
- new net LD3: J1.10 (Pin_10)
- new net V0: J1.3 (Pin_3), RV2.2
Other:
- moved on the sheet: BZ1, RV1, SW1
